Commit message: collision meshes to primitive collision shapes

File: ur_description/urdf/ur10.urdf.xacro (robot description, xacro)
@@ -70,5 +70,6 @@
       <collision>
         <geometry>
-          <mesh filename="package://ur_description/meshes/ur10/collision/base.stl"/>
+          <!-- <mesh filename="package://ur_description/meshes/ur10/collision/base.stl"/> -->
+          <box size="0.2 0.2 0.05"/>
         </geometry>
       </collision>
@@ -101,5 +102,6 @@
       <collision>
         <geometry>
-          <mesh filename="package://ur_description/meshes/ur10/collision/shoulder.stl"/>
+          <!-- <mesh filename="package://ur_description/meshes/ur10/collision/shoulder.stl"/> -->
+          <cylinder radius="0.09" length="0.2"/>
         </geometry>
       </collision>
@@ -131,6 +133,8 @@
       </visual>
       <collision>
-        <geometry>
-          <mesh filename="package://ur_description/meshes/ur10/collision/upperarm.stl"/>
+        <origin xyz="0.0 -0.045 0.3"/>
+        <geometry>
+          <!-- <mesh filename="package://ur_description/meshes/ur10/collision/upperarm.stl"/> -->
+          <cylinder radius="0.09" length="0.8"/>
         </geometry>
       </collision>
@@ -162,6 +166,8 @@
       </visual>
       <collision>
-        <geometry>
-          <mesh filename="package://ur_description/meshes/ur10/collision/forearm.stl"/>
+        <origin xyz="0.0 0.0 0.3"/>
+        <geometry>
+          <!-- <mesh filename="package://ur_description/meshes/ur10/collision/forearm.stl"/> -->
+          <cylinder radius="0.08" length="0.8"/>
         </geometry>
       </collision>
@@ -193,6 +199,8 @@
       </visual>
       <collision>
-        <geometry>
-          <mesh filename="package://ur_description/meshes/ur10/collision/wrist1.stl"/>
+        <origin xyz="0.0 0.11 0.0"/>
+        <geometry>
+          <!-- <mesh filename="package://ur_description/meshes/ur10/collision/wrist1.stl"/> -->
+          <cylinder radius="0.06" length="0.10"/>
         </geometry>
       </collision>
@@ -224,6 +232,8 @@
       </visual>
       <collision>
-        <geometry>
-          <mesh filename="package://ur_description/meshes/ur10/collision/wrist2.stl"/>
+        <origin xyz="0.0 0.0 0.115" rpy="1.5707 0.0 0.0"/>
+        <geometry>
+          <!-- <mesh filename="package://ur_description/meshes/ur10/collision/wrist2.stl"/> -->
+          <cylinder radius="0.058" length="0.13"/>
         </geometry>
       </collision>
@@ -255,6 +265,8 @@
       </visual>
       <collision>
-        <geometry>
-          <mesh filename="package://ur_description/meshes/ur10/collision/wrist3.stl"/>
+        <origin xyz="0.0 0.13 0.0" rpy="1.5707 0.0 0.0"/>
+        <geometry>
+          <!-- <mesh filename="package://ur_description/meshes/ur10/collision/wrist3.stl"/> -->
+          <cylinder radius="0.06" length="0.03"/>
         </geometry>
       </collision>

Commit message: fixed for self collision

File: ur_description/urdf/ur10.urdf.xacro (robot description, xacro)
@@ -103,5 +103,5 @@
         <geometry>
           <!-- <mesh filename="package://ur_description/meshes/ur10/collision/shoulder.stl"/> -->
-          <cylinder radius="0.09" length="0.2"/>
+          <cylinder radius="0.08" length="0.2"/>
         </geometry>
       </collision>
@@ -136,5 +136,5 @@
         <geometry>
           <!-- <mesh filename="package://ur_description/meshes/ur10/collision/upperarm.stl"/> -->
-          <cylinder radius="0.09" length="0.8"/>
+          <cylinder radius="0.07" length="0.8"/>
         </geometry>
       </collision>
@@ -169,5 +169,5 @@
         <geometry>
           <!-- <mesh filename="package://ur_description/meshes/ur10/collision/forearm.stl"/> -->
-          <cylinder radius="0.08" length="0.8"/>
+          <cylinder radius="0.07" length="0.8"/>
         </geometry>
       </collision>
@@ -202,5 +202,5 @@
         <geometry>
           <!-- <mesh filename="package://ur_description/meshes/ur10/collision/wrist1.stl"/> -->
-          <cylinder radius="0.06" length="0.10"/>
+          <cylinder radius="0.05" length="0.10"/>
         </geometry>
       </collision>
@@ -235,5 +235,5 @@
         <geometry>
           <!-- <mesh filename="package://ur_description/meshes/ur10/collision/wrist2.stl"/> -->
-          <cylinder radius="0.058" length="0.13"/>
+          <cylinder radius="0.048" length="0.13"/>
         </geometry>
       </collision>
